File: output.JVCardx4.kicad_pcb (KiCad board)
At the start: 2 copper layers, 344 x 264 mm, 320 parts, among them J6 Conn_02x25_Odd_Even, Q1 mmbt3904, Q2 mmbt3904, Q3 mmbt3904, Q4 mmbt3904, Q5 mmbt3904, Q6 mmbt3904, U1 AMS1117-5.0, U4 SCART_CONN

Commit message: resync
Parts:
- removed the ? at (196.8, 139.8)
- removed the ? at (102.8, 139.8)
- removed the ? at (116.8, 139.8)
- removed the ? at (121.2, 144.2)
- removed the ? at (109.8, 271.2)
- removed the ? at (114.2, 266.8)
- removed the ? at (109.8, 151.2)
- removed the ? at (114.3, 146.8)
- removed the ? at (114.2, 132.8)
- removed the ? at (109.8, 137.2)
- removed the ? at (109.8, 17.2)
- removed the ? at (201.2, 144.2)
- removed the ? at (114.3, 12.8)
- removed the ? at (22.8, 139.8)
- removed the ? at (27.2, 144.2)
- removed the ? at (-57.2, 139.8)
- removed the ? at (-52.8, 144.2)
- removed the ? at (281.2, 144.2)
- removed the ? at (276.8, 139.8)
- removed the ? at (107.2, 144.2)
- removed the C14 at (230.5, 171.5)
- removed the C14 at (-6.50, 246.5)
- removed the C14 at (-6.50, 112.5)
- removed the C14 at (230.5, 37.5)
- removed the C15 at (240.1, 176.0)
- removed the C15 at (-16.1, 242.0)
- removed the C15 at (-16.1, 108.0)
- removed the C15 at (240.1, 42.0)
- removed the C16 at (251.0, 253.0)
- removed the C16 at (-27.0, 165.0)
- removed the C16 at (-27.0, 31.0)
- removed the C16 at (251.0, 119.0)
- removed the C17 at (251.0, 237.0)
- removed the C17 at (-27.0, 181.0)
- removed the C17 at (-27.0, 47.0)
- removed the C17 at (251.0, 103.0)
- removed the C18 at (251.0, 221.0)
- removed the C18 at (-27.0, 197.0)
- removed the C18 at (-27.0, 63.0)
- removed the C18 at (251.0, 87.0)
- removed the C19 at (254.0, 205.0)
- removed the C19 at (-30.0, 213.0)
- removed the C19 at (-30.0, 79.0)
- removed the C19 at (254.0, 71.0)
- removed the C20 at (254.0, 189.0)
- removed the C20 at (-30.0, 229.0)
- removed the C20 at (-30.0, 95.0)
- removed the C20 at (254.0, 55.0)
- removed the C21 at (269.0, 170.0)
- removed the C21 at (-45.0, 248.0)
- removed the C21 at (-45.0, 114.0)
- removed the C21 at (269.0, 36.0)
- removed the C22 at (241.0, 193.0)
- removed the C22 at (-17.0, 225.0)
- removed the C22 at (-17.0, 91.0)
- removed the C22 at (241.0, 59.0)
- removed the C23 at (241.0, 209.0)
- removed the C23 at (-17.0, 209.0)
- removed the C23 at (-17.0, 75.0)
- removed the C23 at (241.0, 75.0)
- removed the C24 at (239.0, 225.0)
- removed the C24 at (-15.0, 193.0)
- removed the C24 at (-15.0, 59.0)
- removed the C24 at (239.0, 91.0)
- removed the C25 at (239.0, 241.0)
- removed the C25 at (-15.0, 177.0)
- removed the C25 at (-15.0, 43.0)
- removed the C25 at (239.0, 107.0)
- removed the C26 at (258.0, 174.0)
- removed the C26 at (-34.0, 244.0)
- removed the C26 at (-34.0, 110.0)
- removed the C26 at (258.0, 40.0)
- removed the C27 at (239.0, 257.0)
- removed the C27 at (-15.0, 161.0)
- removed the C27 at (-15.0, 27.0)
- removed the C27 at (239.0, 123.0)
- removed the D1 at (250.5, 247.0)
- removed the D1 at (-26.5, 171.0)
- removed the D1 at (-26.5, 37.0)
- removed the D1 at (250.5, 113.0)
- removed the D2 at (250.5, 231.0)
- removed the D2 at (-26.5, 187.0)
- removed the D2 at (-26.5, 53.0)
- removed the D2 at (250.5, 97.0)
- removed the D3 at (250.5, 215.0)
- removed the D3 at (-26.5, 203.0)
- removed the D3 at (-26.5, 69.0)
- removed the D3 at (250.5, 81.0)
- removed the D4 at (251.5, 201.0)
- removed the D4 at (-27.5, 217.0)
- removed the D4 at (-27.5, 83.0)
- removed the D4 at (251.5, 67.0)
- removed the D5 at (251.5, 185.0)
- removed the D5 at (-27.5, 233.0)
- removed the D5 at (-27.5, 99.0)
- removed the D5 at (251.5, 51.0)
- removed the D6 at (268.5, 166.0)
- removed the D6 at (-44.5, 252.0)
- removed the D6 at (-44.5, 118.0)
- removed the D6 at (268.5, 32.0)
- removed the H1 at (264.0, 153.5)
- removed the H1 at (-40.0, 264.5)
- removed the H1 at (-40.0, 130.5)
- removed the H1 at (264.0, 19.5)
- removed the H2 at (264.0, 264.5)
- removed the H2 at (-40.0, 153.5)
- removed the H2 at (-40.0, 19.5)
- removed the H2 at (264.0, 130.5)
- removed the J6 at (121.5, 239.5)
- removed the J6 at (102.5, 178.5)
- removed the J6 at (102.5, 44.5)
- removed the J6 at (121.5, 105.5)
- removed the JBlue1 at (266.0, 221.0)
- removed the JBlue1 at (-42.0, 197.0)
- removed the JBlue1 at (-42.0, 63.0)
- removed the JBlue1 at (266.0, 87.0)
- removed the JGreen1 at (266.0, 237.0)
- removed the JGreen1 at (-42.0, 181.0)
- removed the JGreen1 at (-42.0, 47.0)
- removed the JGreen1 at (266.0, 103.0)
- removed the JH1 at (266.0, 205.0)
- removed the JH1 at (-42.0, 213.0)
- removed the JH1 at (-42.0, 79.0)
- removed the JH1 at (266.0, 71.0)
- removed the JLeft1 at (284.0, 170.0)
- removed the JLeft1 at (-60.0, 248.0)
- removed the JLeft1 at (-60.0, 114.0)
- removed the JLeft1 at (284.0, 36.0)
- removed the JRed1 at (266.0, 253.0)
- removed the JRed1 at (-42.0, 165.0)
- removed the JRed1 at (-42.0, 31.0)
- removed the JRed1 at (266.0, 119.0)
- removed the JRight1 at (284.0, 157.0)
- removed the JRight1 at (-60.0, 261.0)
- removed the JRight1 at (-60.0, 127.0)
- removed the JRight1 at (284.0, 23.0)
- removed the JV1 at (266.0, 189.0)
- removed the JV1 at (-42.0, 229.0)
- removed the JV1 at (-42.0, 95.0)
- removed the JV1 at (266.0, 55.0)
- removed the Q1 at (240.0, 254.0)
- removed the Q1 at (-16.0, 164.0)
- removed the Q1 at (-16.0, 30.0)
- removed the Q1 at (240.0, 120.0)
- removed the Q2 at (240.0, 238.0)
- removed the Q2 at (-16.0, 180.0)
- removed the Q2 at (-16.0, 46.0)
- removed the Q2 at (240.0, 104.0)
- removed the Q3 at (240.0, 222.0)
- removed the Q3 at (-16.0, 196.0)
- removed the Q3 at (-16.0, 62.0)
- removed the Q3 at (240.0, 88.0)
- removed the Q4 at (242.0, 206.0)
- removed the Q4 at (-18.0, 212.0)
- removed the Q4 at (-18.0, 78.0)
- removed the Q4 at (242.0, 72.0)
- removed the Q5 at (242.0, 190.0)
- removed the Q5 at (-18.0, 228.0)
- removed the Q5 at (-18.0, 94.0)
- removed the Q5 at (242.0, 56.0)
- removed the Q6 at (259.0, 171.0)
- removed the Q6 at (-35.0, 247.0)
- removed the Q6 at (-35.0, 113.0)
- removed the Q6 at (259.0, 37.0)
- removed the R1 at (234.0, 178.0)
- removed the R1 at (-10.0, 240.0)
- removed the R1 at (-10.0, 106.0)
- removed the R1 at (234.0, 44.0)
- removed the R12 at (258.0, 252.0)
- removed the R12 at (-34.0, 166.0)
- removed the R12 at (-34.0, 32.0)
- removed the R12 at (258.0, 118.0)
- removed the R13 at (258.0, 236.0)
- removed the R13 at (-34.0, 182.0)
- removed the R13 at (-34.0, 48.0)
- removed the R13 at (258.0, 102.0)
- removed the R14 at (258.0, 220.0)
- removed the R14 at (-34.0, 198.0)
- removed the R14 at (-34.0, 64.0)
- removed the R14 at (258.0, 86.0)
- removed the R15 at (258.0, 204.0)
- removed the R15 at (-34.0, 214.0)
- removed the R15 at (-34.0, 80.0)
- removed the R15 at (258.0, 70.0)
- removed the R18 at (258.0, 188.0)
- removed the R18 at (-34.0, 230.0)
- removed the R18 at (-34.0, 96.0)
- removed the R18 at (258.0, 54.0)
- removed the R19 at (244.0, 253.0)
- removed the R19 at (-20.0, 165.0)
- removed the R19 at (-20.0, 31.0)
- removed the R19 at (244.0, 119.0)
- removed the R2 at (234.0, 174.0)
- removed the R2 at (-10.0, 244.0)
- removed the R2 at (-10.0, 110.0)
- removed the R2 at (234.0, 40.0)
- removed the R20 at (244.0, 237.0)
- removed the R20 at (-20.0, 181.0)
- removed the R20 at (-20.0, 47.0)
- removed the R20 at (244.0, 103.0)
- removed the R21 at (244.0, 221.0)
- removed the R21 at (-20.0, 197.0)
- removed the R21 at (-20.0, 63.0)
- removed the R21 at (244.0, 87.0)
- removed the R22 at (246.0, 205.0)
- removed the R22 at (-22.0, 213.0)
- removed the R22 at (-22.0, 79.0)
- removed the R22 at (246.0, 71.0)
- removed the R23 at (246.0, 189.0)
- removed the R23 at (-22.0, 229.0)
- removed the R23 at (-22.0, 95.0)
- removed the R23 at (246.0, 55.0)
- removed the R24 at (263.0, 170.0)
- removed the R24 at (-39.0, 248.0)
- removed the R24 at (-39.0, 114.0)
- removed the R24 at (263.0, 36.0)
- removed the R25 at (244.0, 255.0)
- removed the R25 at (-20.0, 163.0)
- removed the R25 at (-20.0, 29.0)
- removed the R25 at (244.0, 121.0)
- removed the R26 at (244.0, 251.0)
- removed the R26 at (-20.0, 167.0)
- removed the R26 at (-20.0, 33.0)
- removed the R26 at (244.0, 117.0)
- removed the R27 at (244.0, 239.0)
- removed the R27 at (-20.0, 179.0)
- removed the R27 at (-20.0, 45.0)
- removed the R27 at (244.0, 105.0)
- removed the R28 at (244.0, 235.0)
- removed the R28 at (-20.0, 183.0)
- removed the R28 at (-20.0, 49.0)
- removed the R28 at (244.0, 101.0)
- removed the R29 at (244.0, 223.0)
- removed the R29 at (-20.0, 195.0)
- removed the R29 at (-20.0, 61.0)
- removed the R29 at (244.0, 89.0)
- removed the R30 at (244.0, 219.0)
- removed the R30 at (-20.0, 199.0)
- removed the R30 at (-20.0, 65.0)
- removed the R30 at (244.0, 85.0)
- removed the R31 at (246.0, 207.0)
- removed the R31 at (-22.0, 211.0)
- removed the R31 at (-22.0, 77.0)
- removed the R31 at (246.0, 73.0)
- removed the R32 at (246.0, 203.0)
- removed the R32 at (-22.0, 215.0)
- removed the R32 at (-22.0, 81.0)
- removed the R32 at (246.0, 69.0)
- removed the R33 at (246.0, 191.0)
- removed the R33 at (-22.0, 227.0)
- removed the R33 at (-22.0, 93.0)
- removed the R33 at (246.0, 57.0)
- removed the R34 at (246.0, 187.0)
- removed the R34 at (-22.0, 231.0)
- removed the R34 at (-22.0, 97.0)
- removed the R34 at (246.0, 53.0)
- removed the R35 at (263.0, 172.0)
- removed the R35 at (-39.0, 246.0)
- removed the R35 at (-39.0, 112.0)
- removed the R35 at (263.0, 38.0)
- removed the R36 at (263.0, 168.0)
- removed the R36 at (-39.0, 250.0)
- removed the R36 at (-39.0, 116.0)
- removed the R36 at (263.0, 34.0)
- removed the R37 at (240.0, 251.0)
- removed the R37 at (-16.0, 167.0)
- removed the R37 at (-16.0, 33.0)
- removed the R37 at (240.0, 117.0)
- removed the R38 at (240.0, 235.0)
- removed the R38 at (-16.0, 183.0)
- removed the R38 at (-16.0, 49.0)
- removed the R38 at (240.0, 101.0)
- removed the R39 at (240.0, 219.0)
- removed the R39 at (-16.0, 199.0)
- removed the R39 at (-16.0, 65.0)
- removed the R39 at (240.0, 85.0)
- removed the R40 at (242.0, 203.0)
- removed the R40 at (-18.0, 215.0)
- removed the R40 at (-18.0, 81.0)
- removed the R40 at (242.0, 69.0)
- removed the R41 at (242.0, 187.0)
- removed the R41 at (-18.0, 231.0)
- removed the R41 at (-18.0, 97.0)
- removed the R41 at (242.0, 53.0)
- removed the R42 at (259.0, 168.0)
- removed the R42 at (-35.0, 250.0)
- removed the R42 at (-35.0, 116.0)
- removed the R42 at (259.0, 34.0)
- removed the R43 at (236.0, 253.0)
- removed the R43 at (-12.0, 165.0)
- removed the R43 at (-12.0, 31.0)
- removed the R43 at (236.0, 119.0)
- removed the R44 at (236.0, 237.0)
- removed the R44 at (-12.0, 181.0)
- removed the R44 at (-12.0, 47.0)
- removed the R44 at (236.0, 103.0)
- removed the R45 at (236.0, 221.0)
- removed the R45 at (-12.0, 197.0)
- removed the R45 at (-12.0, 63.0)
- removed the R45 at (236.0, 87.0)
- removed the R46 at (238.0, 205.0)
- removed the R46 at (-14.0, 213.0)
- removed the R46 at (-14.0, 79.0)
- removed the R46 at (238.0, 71.0)
- removed the R47 at (238.0, 189.0)
- removed the R47 at (-14.0, 229.0)
- removed the R47 at (-14.0, 95.0)
- removed the R47 at (238.0, 55.0)
- removed the R48 at (255.0, 170.0)
- removed the R48 at (-31.0, 248.0)
- removed the R48 at (-31.0, 114.0)
- removed the R48 at (255.0, 36.0)
- removed the U1 at (228.5, 176.5)
- removed the U1 at (-4.50, 241.5)
- removed the U1 at (-4.50, 107.5)
- removed the U1 at (228.5, 42.5)
- removed the U4 at (280.4, 215.4)
- removed the U4 at (-56.4, 202.6)
- removed the U4 at (-56.4, 68.6)
- removed the U4 at (280.4, 81.4)
- added ?: , holes, F.Cu at (95.5, 142.6)
- added ?: , holes, F.Cu at (100.5, 146.4)
- added ?: , holes, F.Cu at (160.5, 142.6)
- added ?: , holes, F.Cu at (165.5, 146.4)
- added ?: , holes, F.Cu at (30.5, 142.6)
- added ?: , holes, F.Cu at (35.5, 146.4)
- added C14: 10u, Capacitor_SMD:C_0805_2012Metric_Pad1.15x1.40mm_HandSolder, F.Cu at (66.5, 248.5)
- added C14: 10u, Capacitor_SMD:C_0805_2012Metric_Pad1.15x1.40mm_HandSolder, F.Cu at (66.5, 115.5)
- added C15: 47u, Capacitor_SMD:CP_Elec_6.3x7.7, F.Cu at (56.9, 244.0)
- added C15: 47u, Capacitor_SMD:CP_Elec_6.3x7.7, F.Cu at (56.9, 111.0)
- added C16: 47u, Capacitor_SMD:CP_Elec_6.3x7.7, F.Cu at (46.0, 167.0)
- added C16: 47u, Capacitor_SMD:CP_Elec_6.3x7.7, F.Cu at (46.0, 34.0)
- added C17: 47u, Capacitor_SMD:CP_Elec_6.3x7.7, F.Cu at (46.0, 183.0)
- added C17: 47u, Capacitor_SMD:CP_Elec_6.3x7.7, F.Cu at (46.0, 50.0)
- added C18: 47u, Capacitor_SMD:CP_Elec_6.3x7.7, F.Cu at (46.0, 199.0)
- added C18: 47u, Capacitor_SMD:CP_Elec_6.3x7.7, F.Cu at (46.0, 66.0)
- added C19: 10u, Capacitor_SMD:C_0805_2012Metric_Pad1.15x1.40mm_HandSolder, F.Cu at (43.0, 215.0)
- added C19: 10u, Capacitor_SMD:C_0805_2012Metric_Pad1.15x1.40mm_HandSolder, F.Cu at (43.0, 82.0)
- added C20: 10u, Capacitor_SMD:C_0805_2012Metric_Pad1.15x1.40mm_HandSolder, F.Cu at (43.0, 231.0)
- added C20: 10u, Capacitor_SMD:C_0805_2012Metric_Pad1.15x1.40mm_HandSolder, F.Cu at (43.0, 98.0)
- added C21: 10u, Capacitor_SMD:C_0805_2012Metric_Pad1.15x1.40mm_HandSolder, F.Cu at (28.0, 250.0)
- added C21: 10u, Capacitor_SMD:C_0805_2012Metric_Pad1.15x1.40mm_HandSolder, F.Cu at (28.0, 117.0)
- added C22: 1u, Capacitor_SMD:C_0805_2012Metric_Pad1.15x1.40mm_HandSolder, F.Cu at (56.0, 227.0)
- added C22: 1u, Capacitor_SMD:C_0805_2012Metric_Pad1.15x1.40mm_HandSolder, F.Cu at (56.0, 94.0)
- added C23: 1u, Capacitor_SMD:C_0805_2012Metric_Pad1.15x1.40mm_HandSolder, F.Cu at (56.0, 211.0)
- added C23: 1u, Capacitor_SMD:C_0805_2012Metric_Pad1.15x1.40mm_HandSolder, F.Cu at (56.0, 78.0)
- added C24: 1u, Capacitor_SMD:C_0805_2012Metric_Pad1.15x1.40mm_HandSolder, F.Cu at (58.0, 195.0)
- added C24: 1u, Capacitor_SMD:C_0805_2012Metric_Pad1.15x1.40mm_HandSolder, F.Cu at (58.0, 62.0)
- added C25: 1u, Capacitor_SMD:C_0805_2012Metric_Pad1.15x1.40mm_HandSolder, F.Cu at (58.0, 179.0)
- added C25: 1u, Capacitor_SMD:C_0805_2012Metric_Pad1.15x1.40mm_HandSolder, F.Cu at (58.0, 46.0)
- added C26: 1u, Capacitor_SMD:C_0805_2012Metric_Pad1.15x1.40mm_HandSolder, F.Cu at (39.0, 246.0)
- added C26: 1u, Capacitor_SMD:C_0805_2012Metric_Pad1.15x1.40mm_HandSolder, F.Cu at (39.0, 113.0)
- added C27: 1u, Capacitor_SMD:C_0805_2012Metric_Pad1.15x1.40mm_HandSolder, F.Cu at (58.0, 163.0)
- added C27: 1u, Capacitor_SMD:C_0805_2012Metric_Pad1.15x1.40mm_HandSolder, F.Cu at (58.0, 30.0)
- added D1: 7v5, Diode_SMD:D_SOD-123F, F.Cu at (46.5, 173.0)
- added D1: 7v5, Diode_SMD:D_SOD-123F, F.Cu at (46.5, 40.0)
- added D2: 7v5, Diode_SMD:D_SOD-123F, F.Cu at (46.5, 189.0)
- added D2: 7v5, Diode_SMD:D_SOD-123F, F.Cu at (46.5, 56.0)
- added D3: 7v5, Diode_SMD:D_SOD-123F, F.Cu at (46.5, 205.0)
- added D3: 7v5, Diode_SMD:D_SOD-123F, F.Cu at (46.5, 72.0)
- added D4: 7v5, Diode_SMD:D_SOD-123F, F.Cu at (45.5, 219.0)
- added D4: 7v5, Diode_SMD:D_SOD-123F, F.Cu at (45.5, 86.0)
- added D5: 7v5, Diode_SMD:D_SOD-123F, F.Cu at (45.5, 235.0)
- added D5: 7v5, Diode_SMD:D_SOD-123F, F.Cu at (45.5, 102.0)
- added D6: 7v5, Diode_SMD:D_SOD-123F, F.Cu at (28.5, 254.0)
- added D6: 7v5, Diode_SMD:D_SOD-123F, F.Cu at (28.5, 121.0)
- added G***: LOGO, videobits:wakaba, F.Cu at (90.9, 150.4)
- added G***: LOGO, videobits:borgar, F.Cu at (121.6, 211.0)
- added G***: LOGO, videobits:wakaba, F.Cu at (90.9, 17.4)
- added G***: LOGO, videobits:borgar, F.Cu at (121.6, 78.0)
- added H1: MountingHole, MountingHole:MountingHole_3.2mm_M3, F.Cu at (33.0, 266.5)
- added H1: MountingHole, MountingHole:MountingHole_3.2mm_M3, F.Cu at (33.0, 133.5)
- added H2: MountingHole, MountingHole:MountingHole_3.2mm_M3, F.Cu at (33.0, 155.5)
- added H2: MountingHole, MountingHole:MountingHole_3.2mm_M3, F.Cu at (33.0, 22.5)
- added J6: Conn_02x25_Odd_Even, Connector_PinHeader_2.54mm:PinHeader_2x25_P2.54mm_Horizontal, F.Cu at (175.5, 180.5)
- added J6: Conn_02x25_Odd_Even, Connector_PinHeader_2.54mm:PinHeader_2x25_P2.54mm_Horizontal, F.Cu at (175.5, 47.5)
- added JBlue1: Conn_Coaxial, videobits:BNC_Amphenol_B6252HB-NPP3G-50_Horizontal_smallerpads, F.Cu at (31.0, 199.0)
- added JBlue1: Conn_Coaxial, videobits:BNC_Amphenol_B6252HB-NPP3G-50_Horizontal_smallerpads, F.Cu at (31.0, 66.0)
- added JGreen1: Conn_Coaxial, videobits:BNC_Amphenol_B6252HB-NPP3G-50_Horizontal_smallerpads, F.Cu at (31.0, 183.0)
- added JGreen1: Conn_Coaxial, videobits:BNC_Amphenol_B6252HB-NPP3G-50_Horizontal_smallerpads, F.Cu at (31.0, 50.0)
- added JH1: Conn_Coaxial, videobits:BNC_Amphenol_B6252HB-NPP3G-50_Horizontal_smallerpads, F.Cu at (31.0, 215.0)
- added JH1: Conn_Coaxial, videobits:BNC_Amphenol_B6252HB-NPP3G-50_Horizontal_smallerpads, F.Cu at (31.0, 82.0)
- added JLeft1: Conn_Coaxial, videobits:Cheapo_RCA_single_edge, F.Cu at (13.0, 250.0)
- added JLeft1: Conn_Coaxial, videobits:Cheapo_RCA_single_edge, F.Cu at (13.0, 117.0)
- added JRed1: Conn_Coaxial, videobits:BNC_Amphenol_B6252HB-NPP3G-50_Horizontal_smallerpads, F.Cu at (31.0, 167.0)
- added JRed1: Conn_Coaxial, videobits:BNC_Amphenol_B6252HB-NPP3G-50_Horizontal_smallerpads, F.Cu at (31.0, 34.0)
- added JRight1: Conn_Coaxial, videobits:Cheapo_RCA_single_edge, F.Cu at (13.0, 263.0)
- added JRight1: Conn_Coaxial, videobits:Cheapo_RCA_single_edge, F.Cu at (13.0, 130.0)
- added JV1: Conn_Coaxial, videobits:BNC_Amphenol_B6252HB-NPP3G-50_Horizontal_smallerpads, F.Cu at (31.0, 231.0)
- added JV1: Conn_Coaxial, videobits:BNC_Amphenol_B6252HB-NPP3G-50_Horizontal_smallerpads, F.Cu at (31.0, 98.0)
- added Q1: mmbt3904, Package_TO_SOT_SMD:SOT-23, F.Cu at (57.0, 166.0)
- added Q1: mmbt3904, Package_TO_SOT_SMD:SOT-23, F.Cu at (57.0, 33.0)
- added Q2: mmbt3904, Package_TO_SOT_SMD:SOT-23, F.Cu at (57.0, 182.0)
- added Q2: mmbt3904, Package_TO_SOT_SMD:SOT-23, F.Cu at (57.0, 49.0)
- added Q3: mmbt3904, Package_TO_SOT_SMD:SOT-23, F.Cu at (57.0, 198.0)
- added Q3: mmbt3904, Package_TO_SOT_SMD:SOT-23, F.Cu at (57.0, 65.0)
- added Q4: mmbt3904, Package_TO_SOT_SMD:SOT-23, F.Cu at (55.0, 214.0)
- added Q4: mmbt3904, Package_TO_SOT_SMD:SOT-23, F.Cu at (55.0, 81.0)
- added Q5: mmbt3904, Package_TO_SOT_SMD:SOT-23, F.Cu at (55.0, 230.0)
- added Q5: mmbt3904, Package_TO_SOT_SMD:SOT-23, F.Cu at (55.0, 97.0)
- added Q6: mmbt3904, Package_TO_SOT_SMD:SOT-23, F.Cu at (38.0, 249.0)
- added Q6: mmbt3904, Package_TO_SOT_SMD:SOT-23, F.Cu at (38.0, 116.0)
- added R1: 1k, Resistor_SMD:R_0805_2012Metric_Pad1.15x1.40mm_HandSolder, F.Cu at (63.0, 242.0)
- added R1: 1k, Resistor_SMD:R_0805_2012Metric_Pad1.15x1.40mm_HandSolder, F.Cu at (63.0, 109.0)
- added R12: 75, Resistor_SMD:R_0805_2012Metric_Pad1.15x1.40mm_HandSolder, F.Cu at (39.0, 168.0)
- added R12: 75, Resistor_SMD:R_0805_2012Metric_Pad1.15x1.40mm_HandSolder, F.Cu at (39.0, 35.0)
- added R13: 75, Resistor_SMD:R_0805_2012Metric_Pad1.15x1.40mm_HandSolder, F.Cu at (39.0, 184.0)
- added R13: 75, Resistor_SMD:R_0805_2012Metric_Pad1.15x1.40mm_HandSolder, F.Cu at (39.0, 51.0)
- added R14: 75, Resistor_SMD:R_0805_2012Metric_Pad1.15x1.40mm_HandSolder, F.Cu at (39.0, 200.0)
- added R14: 75, Resistor_SMD:R_0805_2012Metric_Pad1.15x1.40mm_HandSolder, F.Cu at (39.0, 67.0)
- added R15: 75, Resistor_SMD:R_0805_2012Metric_Pad1.15x1.40mm_HandSolder, F.Cu at (39.0, 216.0)
- added R15: 75, Resistor_SMD:R_0805_2012Metric_Pad1.15x1.40mm_HandSolder, F.Cu at (39.0, 83.0)
- added R18: 75, Resistor_SMD:R_0805_2012Metric_Pad1.15x1.40mm_HandSolder, F.Cu at (39.0, 232.0)
- added R18: 75, Resistor_SMD:R_0805_2012Metric_Pad1.15x1.40mm_HandSolder, F.Cu at (39.0, 99.0)
- added R19: 100, Resistor_SMD:R_0805_2012Metric_Pad1.15x1.40mm_HandSolder, F.Cu at (53.0, 167.0)
- added R19: 100, Resistor_SMD:R_0805_2012Metric_Pad1.15x1.40mm_HandSolder, F.Cu at (53.0, 34.0)
- added R2: 1k, Resistor_SMD:R_0805_2012Metric_Pad1.15x1.40mm_HandSolder, F.Cu at (63.0, 246.0)
- added R2: 1k, Resistor_SMD:R_0805_2012Metric_Pad1.15x1.40mm_HandSolder, F.Cu at (63.0, 113.0)
- added R20: 100, Resistor_SMD:R_0805_2012Metric_Pad1.15x1.40mm_HandSolder, F.Cu at (53.0, 183.0)
- added R20: 100, Resistor_SMD:R_0805_2012Metric_Pad1.15x1.40mm_HandSolder, F.Cu at (53.0, 50.0)
- added R21: 100, Resistor_SMD:R_0805_2012Metric_Pad1.15x1.40mm_HandSolder, F.Cu at (53.0, 199.0)
- added R21: 100, Resistor_SMD:R_0805_2012Metric_Pad1.15x1.40mm_HandSolder, F.Cu at (53.0, 66.0)
- added R22: 100, Resistor_SMD:R_0805_2012Metric_Pad1.15x1.40mm_HandSolder, F.Cu at (51.0, 215.0)
- added R22: 100, Resistor_SMD:R_0805_2012Metric_Pad1.15x1.40mm_HandSolder, F.Cu at (51.0, 82.0)
- added R23: 100, Resistor_SMD:R_0805_2012Metric_Pad1.15x1.40mm_HandSolder, F.Cu at (51.0, 231.0)
- added R23: 100, Resistor_SMD:R_0805_2012Metric_Pad1.15x1.40mm_HandSolder, F.Cu at (51.0, 98.0)
- added R24: 100, Resistor_SMD:R_0805_2012Metric_Pad1.15x1.40mm_HandSolder, F.Cu at (34.0, 250.0)
- added R24: 100, Resistor_SMD:R_0805_2012Metric_Pad1.15x1.40mm_HandSolder, F.Cu at (34.0, 117.0)
- added R25: 56k, Resistor_SMD:R_0805_2012Metric_Pad1.15x1.40mm_HandSolder, F.Cu at (53.0, 165.0)
- added R25: 56k, Resistor_SMD:R_0805_2012Metric_Pad1.15x1.40mm_HandSolder, F.Cu at (53.0, 32.0)
- added R26: 33k, Resistor_SMD:R_0805_2012Metric_Pad1.15x1.40mm_HandSolder, F.Cu at (53.0, 169.0)
- added R26: 33k, Resistor_SMD:R_0805_2012Metric_Pad1.15x1.40mm_HandSolder, F.Cu at (53.0, 36.0)
- added R27: 56k, Resistor_SMD:R_0805_2012Metric_Pad1.15x1.40mm_HandSolder, F.Cu at (53.0, 181.0)
- added R27: 56k, Resistor_SMD:R_0805_2012Metric_Pad1.15x1.40mm_HandSolder, F.Cu at (53.0, 48.0)
- added R28: 33k, Resistor_SMD:R_0805_2012Metric_Pad1.15x1.40mm_HandSolder, F.Cu at (53.0, 185.0)
- added R28: 33k, Resistor_SMD:R_0805_2012Metric_Pad1.15x1.40mm_HandSolder, F.Cu at (53.0, 52.0)
- added R29: 56k, Resistor_SMD:R_0805_2012Metric_Pad1.15x1.40mm_HandSolder, F.Cu at (53.0, 197.0)
- added R29: 56k, Resistor_SMD:R_0805_2012Metric_Pad1.15x1.40mm_HandSolder, F.Cu at (53.0, 64.0)
- added R30: 33k, Resistor_SMD:R_0805_2012Metric_Pad1.15x1.40mm_HandSolder, F.Cu at (53.0, 201.0)
- added R30: 33k, Resistor_SMD:R_0805_2012Metric_Pad1.15x1.40mm_HandSolder, F.Cu at (53.0, 68.0)
- added R31: 33k, Resistor_SMD:R_0805_2012Metric_Pad1.15x1.40mm_HandSolder, F.Cu at (51.0, 213.0)
- added R31: 33k, Resistor_SMD:R_0805_2012Metric_Pad1.15x1.40mm_HandSolder, F.Cu at (51.0, 80.0)
- added R32: 33k, Resistor_SMD:R_0805_2012Metric_Pad1.15x1.40mm_HandSolder, F.Cu at (51.0, 217.0)
- added R32: 33k, Resistor_SMD:R_0805_2012Metric_Pad1.15x1.40mm_HandSolder, F.Cu at (51.0, 84.0)
- added R33: 33k, Resistor_SMD:R_0805_2012Metric_Pad1.15x1.40mm_HandSolder, F.Cu at (51.0, 229.0)
- added R33: 33k, Resistor_SMD:R_0805_2012Metric_Pad1.15x1.40mm_HandSolder, F.Cu at (51.0, 96.0)
- added R34: 33k, Resistor_SMD:R_0805_2012Metric_Pad1.15x1.40mm_HandSolder, F.Cu at (51.0, 233.0)
- added R34: 33k, Resistor_SMD:R_0805_2012Metric_Pad1.15x1.40mm_HandSolder, F.Cu at (51.0, 100.0)
- added R35: 33k, Resistor_SMD:R_0805_2012Metric_Pad1.15x1.40mm_HandSolder, F.Cu at (34.0, 248.0)
- added R35: 33k, Resistor_SMD:R_0805_2012Metric_Pad1.15x1.40mm_HandSolder, F.Cu at (34.0, 115.0)
- added R36: 33k, Resistor_SMD:R_0805_2012Metric_Pad1.15x1.40mm_HandSolder, F.Cu at (34.0, 252.0)
- added R36: 33k, Resistor_SMD:R_0805_2012Metric_Pad1.15x1.40mm_HandSolder, F.Cu at (34.0, 119.0)
- added R37: 390, Resistor_SMD:R_0805_2012Metric_Pad1.15x1.40mm_HandSolder, F.Cu at (57.0, 169.0)
- added R37: 390, Resistor_SMD:R_0805_2012Metric_Pad1.15x1.40mm_HandSolder, F.Cu at (57.0, 36.0)
- added R38: 390, Resistor_SMD:R_0805_2012Metric_Pad1.15x1.40mm_HandSolder, F.Cu at (57.0, 185.0)
- added R38: 390, Resistor_SMD:R_0805_2012Metric_Pad1.15x1.40mm_HandSolder, F.Cu at (57.0, 52.0)
- added R39: 390, Resistor_SMD:R_0805_2012Metric_Pad1.15x1.40mm_HandSolder, F.Cu at (57.0, 201.0)
- added R39: 390, Resistor_SMD:R_0805_2012Metric_Pad1.15x1.40mm_HandSolder, F.Cu at (57.0, 68.0)
- added R40: 2k7, Resistor_SMD:R_0805_2012Metric_Pad1.15x1.40mm_HandSolder, F.Cu at (55.0, 217.0)
- added R40: 2k7, Resistor_SMD:R_0805_2012Metric_Pad1.15x1.40mm_HandSolder, F.Cu at (55.0, 84.0)
- added R41: 2k7, Resistor_SMD:R_0805_2012Metric_Pad1.15x1.40mm_HandSolder, F.Cu at (55.0, 233.0)
- added R41: 2k7, Resistor_SMD:R_0805_2012Metric_Pad1.15x1.40mm_HandSolder, F.Cu at (55.0, 100.0)
- added R42: 2k7, Resistor_SMD:R_0805_2012Metric_Pad1.15x1.40mm_HandSolder, F.Cu at (38.0, 252.0)
- added R42: 2k7, Resistor_SMD:R_0805_2012Metric_Pad1.15x1.40mm_HandSolder, F.Cu at (38.0, 119.0)
- added R43: 100, Resistor_SMD:R_0805_2012Metric_Pad1.15x1.40mm_HandSolder, F.Cu at (61.0, 167.0)
- added R43: 100, Resistor_SMD:R_0805_2012Metric_Pad1.15x1.40mm_HandSolder, F.Cu at (61.0, 34.0)
- added R44: 100, Resistor_SMD:R_0805_2012Metric_Pad1.15x1.40mm_HandSolder, F.Cu at (61.0, 183.0)
- added R44: 100, Resistor_SMD:R_0805_2012Metric_Pad1.15x1.40mm_HandSolder, F.Cu at (61.0, 50.0)
- added R45: 100, Resistor_SMD:R_0805_2012Metric_Pad1.15x1.40mm_HandSolder, F.Cu at (61.0, 199.0)
- added R45: 100, Resistor_SMD:R_0805_2012Metric_Pad1.15x1.40mm_HandSolder, F.Cu at (61.0, 66.0)
- added R46: 100, Resistor_SMD:R_0805_2012Metric_Pad1.15x1.40mm_HandSolder, F.Cu at (59.0, 215.0)
- added R46: 100, Resistor_SMD:R_0805_2012Metric_Pad1.15x1.40mm_HandSolder, F.Cu at (59.0, 82.0)
- added R47: 100, Resistor_SMD:R_0805_2012Metric_Pad1.15x1.40mm_HandSolder, F.Cu at (59.0, 231.0)
- added R47: 100, Resistor_SMD:R_0805_2012Metric_Pad1.15x1.40mm_HandSolder, F.Cu at (59.0, 98.0)
- added R48: 100, Resistor_SMD:R_0805_2012Metric_Pad1.15x1.40mm_HandSolder, F.Cu at (42.0, 250.0)
- added R48: 100, Resistor_SMD:R_0805_2012Metric_Pad1.15x1.40mm_HandSolder, F.Cu at (42.0, 117.0)
- added U1: AMS1117-5.0, Package_TO_SOT_SMD:SOT-223-3_TabPin2, F.Cu at (68.5, 243.5)
- added U1: AMS1117-5.0, Package_TO_SOT_SMD:SOT-223-3_TabPin2, F.Cu at (68.5, 110.5)
- added U4: SCART_CONN, custom_components:SCART_CONN, F.Cu at (16.6, 204.6)
- added U4: SCART_CONN, custom_components:SCART_CONN, F.Cu at (16.6, 71.6)
Routing:
- net (no net): track 3501.6 -> 1750.8 mm, vias 382 -> 191
- net /Vs: track 400.7 -> 200.4 mm, vias 2 -> 1
- net /Cs: track 378.6 -> 189.3 mm, vias 2 -> 1
- net +12V: track 362.3 -> 181.1 mm, vias 12 -> 6
- net /Bo: track 335.8 -> 167.9 mm, vias 2 -> 1
- net /Audio: track 319.9 -> 160.0 mm
- net /Ro: track 314.7 -> 157.3 mm
- net /Go: track 314.2 -> 157.1 mm
- net +15V: track 272.8 -> 136.4 mm
- net /Hi: track 128.5 -> 64.3 mm
- net Net-(JRight1-Pad1): track 124.4 -> 62.2 mm
- net /Ai: track 120.9 -> 60.5 mm
- net /Ri: track 65.9 -> 32.9 mm
- net /Gi: track 46.9 -> 23.5 mm
- net /Bi: track 46.4 -> 23.2 mm
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Other:
- board size 344 x 264 mm -> 170 x 263 mm

Commit message: new gerbers for BNC and SCART hole plates
Other:
- net class Default removed
